File: electronics/dual_driver.sch (KiCad schematic (older format))
At the start: 26 parts, among them J1 Screw_Terminal_01x02, J2 Conn_01x02_Female, J3 Conn_01x02_Female, J4 Screw_Terminal_01x02, J5 Screw_Terminal_01x02, Q1 IRF540N, Q2 IRF540N, U1 LM358

Commit message: Added trimpots to schematic
Parts:
- added RV? (x2): POT_TRIM_1k, symbol POT_TRIM
- R15, R16, R3, R4: value 1k -> 5k6
Connections:
- new net: RV?.2, U1.3 (+)
- new net: RV?.2, U1.5 (+)
- new net: R3.2, RV?.1
- new net: R4.1, RV?.3
- new net: R15.2, RV?.1
- new net: R16.1, RV?.3
Changed lines of the file:
@@
 P 3050 3050
 F 0 "R3" V 3130 3050 50  0000 C CNN
-F 1 "1k" V 3050 3050 50  0000 C CNN
+F 1 "5k6" V 3050 3050 50  0000 C CNN
 F 2 "Resistors_THT:R_Axial_DIN0516_L15.5mm_D5.0mm_P20.32mm_Horizontal" V 2980 3050 50  0001 C CNN
 F 3 "" H 3050 3050 50  0001 C CNN
@@
 P 3050 4600
 F 0 "R4" V 3130 4600 50  0000 C CNN
-F 1 "1k" V 3050 4600 50  0000 C CNN
+F 1 "5k6" V 3050 4600 50  0000 C CNN
 F 2 "Resistors_THT:R_Axial_DIN0516_L15.5mm_D5.0mm_P20.32mm_Horizontal" V 2980 4600 50  0001 C CNN
 F 3 "" H 3050 4600 50  0001 C CNN
@@
 P 8000 3000
 F 0 "R15" V 8080 3000 50  0000 C CNN
-F 1 "1k" V 8000 3000 50  0000 C CNN
+F 1 "5k6" V 8000 3000 50  0000 C CNN
 F 2 "Resistors_THT:R_Axial_DIN0516_L15.5mm_D5.0mm_P20.32mm_Horizontal" V 7930 3000 50  0001 C CNN
 F 3 "" H 8000 3000 50  0001 C CNN
@@
 P 8000 4600
 F 0 "R16" V 8080 4600 50  0000 C CNN
-F 1 "1k" V 8000 4600 50  0000 C CNN
+F 1 "5k6" V 8000 4600 50  0000 C CNN
 F 2 "Resistors_THT:R_Axial_DIN0516_L15.5mm_D5.0mm_P20.32mm_Horizontal" V 7930 4600 50  0001 C CNN
 F 3 "" H 8000 4600 50  0001 C CNN
@@
 Connection ~ 3050 5150
 Wire Wire Line
-	3050 3200 3050 4450
-Wire Wire Line
 	3050 4750 3050 5150
 Wire Wire Line
@@
 Connection ~ 6200 3850
 Wire Wire Line
-	3300 3750 3050 3750
-Connection ~ 3050 3750
-Wire Wire Line
 	3300 3950 2600 3950
 Connection ~ 2600 3950
@@
 	6950 4150 6950 5150
 Connection ~ 6950 5150
-Wire Wire Line
-	8000 3150 8000 4450
 Wire Wire Line
 	8000 2150 8000 2850
@@
 Wire Wire Line
 	7850 2250 8000 2250
-Wire Wire Line
-	7150 3750 8000 3750
-Connection ~ 8000 3750
 Wire Wire Line
 	6700 3450 7500 3450
@@
 Wire Wire Line
 	9900 2750 9900 2850
+$Comp
+L POT_TRIM RV?
+U 1 1 5AB380F0
+P 8000 3750
+F 0 "RV?" V 7825 3750 50  0000 C CNN
+F 1 "POT_TRIM_1k" V 7900 3750 50  0000 C CNN
+F 2 "" H 8000 3750 50  0001 C CNN
+F 3 "" H 8000 3750 50  0001 C CNN
+	1    8000 3750
+	-1   0    0    -1
+$EndComp
+$Comp
+L POT_TRIM RV?
+U 1 1 5AB381F0
+P 3050 3750
+F 0 "RV?" V 2875 3750 50  0000 C CNN
+F 1 "POT_TRIM_1k" V 2950 3750 50  0000 C CNN
+F 2 "" H 3050 3750 50  0001 C CNN
+F 3 "" H 3050 3750 50  0001 C CNN
+	1    3050 3750
+	1    0    0    -1
+$EndComp
+Wire Wire Line
+	3050 3200 3050 3600
+Wire Wire Line
+	3050 3900 3050 4450
+Wire Wire Line
+	3300 3750 3200 3750
+Wire Wire Line
+	7150 3750 7850 3750
+Wire Wire Line
+	8000 3150 8000 3600
+Wire Wire Line
+	8000 3900 8000 4450
 $EndSCHEMATC
